File: Version 1.1/Hardware/PIC10F200 PCB.kicad_pcb (KiCad board)
At the start: 2 copper layers, 42 x 42 mm, 14 parts, among them J1 Conn_01x06_Female, SW1 SW_DPST_x2, SW2 SW_DPST_x2, U1 PIC10F200-IP

Commit message: Add Version 1.1 and Version 2.1, Update README.md
Parts:
- R1, R2, R3, R4: footprint Resistor_THT:R_Axial_DIN0207_L6.3mm_D2.5mm_P10.16mm_Horizontal -> Resistor_THT:R_Axial_DIN0309_L9.0mm_D3.2mm_P15.24mm_Horizontal
- moved R2 11.7 mm to (150.4, 100.6)
- moved R1 5.58 mm to (138.8, 85.4)
- moved R3 3.68 mm to (139.6, 77.0)
- moved D1 2.20 mm to (145.8, 88.4)
- moved D2 2.20 mm to (145.7, 98.0)
- moved R4 1.90 mm to (124.4, 109.0)
Routing:
- net GP2: track 13.4 -> 23.7 mm
- net Net-(D2-Pad2): track 6.06 -> 15.6 mm
- net GP1: track 41.2 -> 32.9 mm
- net Net-(D1-Pad2): track 6.32 -> 14.1 mm
- net Net-(R3-Pad2): track 0.00 -> 6.15 mm
- net Net-(R4-Pad2): track 9.96 -> 13.8 mm
- net VSS: track 148.6 -> 151.5 mm
- net GP0: track 25.9 -> 28.4 mm
