File: Hardware/Version 1.2/Hardware/PIC10F200 PCB.kicad_pcb (KiCad board)
At the start: 2 copper layers, 45 x 45 mm, 14 parts, among them J1 Conn_01x06_Female, SW1 SW_DPST_x2, SW2 SW_DPST_x2, U1 PIC10F200-IP

Commit message: Added and Updated all Files
Other:
- board text added: "PCB Way"
- board text added: "Ver. 1.2"
Changed lines of the file:
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@@
       (drillshape 0)
       (scaleselection 1)
-      (outputdirectory "D:/")
+      (outputdirectory "../Fabrication/PCB Way/")
     )
   )
@@
   (gr_line (start 111 111) (end 111 78) (layer "Edge.Cuts") (width 0.1))
   (gr_line (start 156 78) (end 156 111) (layer "Edge.Cuts") (width 0.1))
+  (gr_text "Ver. 1.2" (at 152.4 93.940225 90) (layer "B.SilkS")
+    (effects (font (size 1 1) (thickness 0.15)) (justify mirror))
+  )
+  (gr_text "PCB Way" (at 149.86 93.98 90) (layer "B.SilkS")
+    (effects (font (size 1 1) (thickness 0.15)) (justify mirror))
+  )
+  (gr_text "PCB Way" (at 116.84 104.14) (layer "F.SilkS")
+    (effects (font (size 1.5 1.5) (thickness 0.3)))
+  )
+  (gr_text "Ver. 1.2" (at 147.32 104) (layer "F.SilkS")
+    (effects (font (size 1.5 1.5) (thickness 0.3)))
+  )
   (segment (start 145 86.38) (end 145 81.46) (width 0.5) (layer "F.Cu") (net 2))
   (segment (start 145 81.46) (end 141.54 78) (width 0.5) (layer "F.Cu") (net 2))
